File: hardware/sensor/currentSource.kicad_sch (KiCad schematic)
At the start: 0 parts

Commit message: commit to save work from misbehaving laptop
Parts:
- added Q? (x2): BC847BDW1, Package_TO_SOT_SMD:SOT-363_SC-70-6, symbol Transistor_BJT:BC847BDW1
- added R?: 4k7, symbol Device:R
Connections:
- net In: now also Q?.6 (C1)
- new net: Q?.1 (E1), R?.1
- new net GND: R?.2
Changed lines of the file:
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@@
 (kicad_sch (version 20230121) (generator eeschema)
   (paper "A5")
-  (hierarchical_label "In" (shape input) (at 88.9 50.8 0) (fields_autoplaced)
+  (wire (pts (xy 102.87 78.74) (xy 102.87 81.28))
+    (stroke (width 0) (type default))
+  )
+  (wire (pts (xy 102.87 66.04) (xy 102.87 71.12))
+    (stroke (width 0) (type default))
+  )
+  (wire (pts (xy 100.965 50.165) (xy 102.87 50.165))
+    (stroke (width 0) (type default))
+  )
+  (wire (pts (xy 102.87 50.165) (xy 102.87 55.88))
+    (stroke (width 0) (type default))
+  )
+  (hierarchical_label "In" (shape input) (at 100.965 50.165 180) (fields_autoplaced)
+    (effects (font (size 1.27 1.27)) (justify right))
+  )
+  (hierarchical_label "V_{DD}" (shape input) (at 33.655 66.04 0) (fields_autoplaced)
     (effects (font (size 1.27 1.27)) (justify left))
   )
-  (hierarchical_label "Out" (shape input) (at 88.9 63.5 0) (fields_autoplaced)
-    (effects (font (size 1.27 1.27)) (justify left))
+  (symbol (lib_id "Transistor_BJT:BC847BDW1") (at 34.29 86.995 0) (unit 2)
+    (in_bom yes) (on_board yes) (dnp no) (fields_autoplaced)
+    (property "Reference" "Q?" (at 40.005 85.725 0)
+      (effects (font (size 1.27 1.27)) (justify left))
+    )
+    (property "Value" "BC847BDW1" (at 40.005 88.265 0)
+      (effects (font (size 1.27 1.27)) (justify left))
+    )
+    (property "Footprint" "Package_TO_SOT_SMD:SOT-363_SC-70-6" (at 39.37 84.455 0)
+      (effects (font (size 1.27 1.27)) hide)
+    )
+    (property "Datasheet" "http://www.onsemi.com/pub_link/Collateral/BC846BDW1T1-D.PDF" (at 34.29 86.995 0)
+      (effects (font (size 1.27 1.27)) hide)
+    )
+    (pin "6")
+    (pin "5")
+    (pin "1")
+    (pin "3")
+    (pin "2")
+    (pin "4")
+    (instances
+      (project "sensor"
+        (path "/867f520a-eae4-4e8b-a296-c3a5e3f80a59/5d2941c3-72f3-42b8-875e-cd68d6b4d80f/793e8ff2-2956-4227-9407-3cc0bcbe3d99"
+          (reference "Q?") (unit 2)
+        )
+      )
+    )
   )
-  (hierarchical_label "V_{DD}" (shape input) (at 76.2 50.8 0) (fields_autoplaced)
-    (effects (font (size 1.27 1.27)) (justify left))
+  (symbol (lib_id "Device:R") (at 102.87 74.93 0) (unit 1)
+    (in_bom yes) (on_board yes) (dnp no) (fields_autoplaced)
+    (property "Reference" "R?" (at 105.41 73.66 0)
+      (effects (font (size 1.27 1.27)) (justify left))
+    )
+    (property "Value" "4k7" (at 105.41 76.2 0)
+      (effects (font (size 1.27 1.27)) (justify left))
+    )
+    (property "Footprint" "" (at 101.092 74.93 90)
+      (effects (font (size 1.27 1.27)) hide)
+    )
+    (property "Datasheet" "~" (at 102.87 74.93 0)
+      (effects (font (size 1.27 1.27)) hide)
+    )
+    (pin "2")
+    (pin "1")
+    (instances
+      (project "sensor"
+        (path "/867f520a-eae4-4e8b-a296-c3a5e3f80a59/5d2941c3-72f3-42b8-875e-cd68d6b4d80f/793e8ff2-2956-4227-9407-3cc0bcbe3d99"
+          (reference "R?") (unit 1)
+        )
+      )
+    )
+  )
+  (symbol (lib_id "power:GND") (at 102.87 81.28 0) (unit 1)
+    (in_bom yes) (on_board yes) (dnp no) (fields_autoplaced)
+    (property "Reference" "#PWR05" (at 102.87 87.63 0)
+      (effects (font (size 1.27 1.27)) hide)
+    )
+    (property "Value" "GND" (at 102.87 85.725 0)
+      (effects (font (size 1.27 1.27)))
+    )
+    (property "Footprint" "" (at 102.87 81.28 0)
+      (effects (font (size 1.27 1.27)) hide)
+    )
+    (property "Datasheet" "" (at 102.87 81.28 0)
+      (effects (font (size 1.27 1.27)) hide)
+    )
+    (pin "1")
+    (instances
+      (project "sensor"
+        (path "/867f520a-eae4-4e8b-a296-c3a5e3f80a59/25ef8c17-2fa6-41c6-9d65-771e7f962afe"
+          (reference "#PWR05") (unit 1)
+        )
+        (path "/867f520a-eae4-4e8b-a296-c3a5e3f80a59/5d2941c3-72f3-42b8-875e-cd68d6b4d80f/793e8ff2-2956-4227-9407-3cc0bcbe3d99"
+          (reference "#PWR012") (unit 1)
+        )
+      )
+    )
+  )
+  (symbol (lib_id "Transistor_BJT:BC847BDW1") (at 100.33 60.96 0) (unit 1)
+    (in_bom yes) (on_board yes) (dnp no) (fields_autoplaced)
+    (property "Reference" "Q?" (at 106.045 59.69 0)
+      (effects (font (size 1.27 1.27)) (justify left))
+    )
+    (property "Value" "BC847BDW1" (at 106.045 62.23 0)
+      (effects (font (size 1.27 1.27)) (justify left))
+    )
+    (property "Footprint" "Package_TO_SOT_SMD:SOT-363_SC-70-6" (at 105.41 58.42 0)
+      (effects (font (size 1.27 1.27)) hide)
+    )
+    (property "Datasheet" "http://www.onsemi.com/pub_link/Collateral/BC846BDW1T1-D.PDF" (at 100.33 60.96 0)
+      (effects (font (size 1.27 1.27)) hide)
+    )
+    (pin "6")
+    (pin "5")
+    (pin "1")
+    (pin "3")
+    (pin "2")
+    (pin "4")
+    (instances
+      (project "sensor"
+        (path "/867f520a-eae4-4e8b-a296-c3a5e3f80a59/5d2941c3-72f3-42b8-875e-cd68d6b4d80f/793e8ff2-2956-4227-9407-3cc0bcbe3d99"
+          (reference "Q?") (unit 1)
+        )
+      )
+    )
   )
 )
