File: hardware/sensor/sensor.kicad_pcb (KiCad board)
At the start: 4 copper layers, 40 x 50 mm, 65 parts, among them J101 Conn_Coaxial, J201 PWR, J202 control signals, J203 GND, J204 LDO_{EN}, J205 V_{DD}AN, J206 V_{DD}MCU, J207 GND, J208 GND, J301 U_{ref}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

Commit message: Add bom and final version of rev 1.0
Parts:
- added D601: RED, Diode_SMD:D_0805_2012Metric_Pad1.15x1.40mm_HandSolder, F.Cu at (146.8, 106.5)
- added D602: GREEN, Diode_SMD:D_0805_2012Metric_Pad1.15x1.40mm_HandSolder, F.Cu at (144.5, 106.5)
- added R602: 5k1, Resistor_SMD:R_0805_2012Metric_Pad1.20x1.40mm_HandSolder, F.Cu at (140.2, 106.0)
- added R603: 5k1, Resistor_SMD:R_0805_2012Metric_Pad1.20x1.40mm_HandSolder, F.Cu at (140.2, 108.0)
- J601: footprint Connector:Tag-Connect_TC2030-IDC-NL_2x03_P1.27mm_Vertical -> Connector:Tag-Connect_TC2030-IDC-FP_2x03_P1.27mm_Vertical
- moved J601 1.42 mm to (126.6, 96.8)
- moved J203 0.56 mm to (141.2, 104.2)
Routing:
- net Net-(D601-K): track 0.00 -> 7.10 mm
- net /Microcontroller/io_p025: track 16.4 -> 22.6 mm, vias 0 -> 2
- net /Microcontroller/swd_clk: track 9.43 -> 15.3 mm
- net Net-(D602-K): track 0.00 -> 4.47 mm
- net /Microcontroller/swd_rst: track 26.0 -> 30.0 mm
- net GND: track 69.3 -> 73.1 mm, vias 36 -> 148
- net /Microcontroller/io_p024: track 22.2 -> 25.8 mm
- net /Microcontroller/swd_io: track 6.29 -> 7.96 mm
- net /Microcontroller/LDO_{EN}: track 30.0 -> 31.3 mm
- net /Microcontroller/V_{DD}: track 21.9 -> 23.0 mm
- net /P_{IN}/EH-ON: vias 1 -> 2
- net /P_{IN}/PWG-Vout: vias 1 -> 2
- net /P_{IN}/PWG-LDO: vias 1 -> 2
- net /P_{IN}/HBO-MCU: vias 1 -> 2
Other:
- board text added: "LDO_{out} gnd x 2 V_{DD}"
